File: colordance_mini.kicad_pcb (KiCad board)
At the start: 2 copper layers, 180 x 125 mm, 75 parts, among them J1 XLR3, J10 CONN_01X06, J11 CONN_01X04, J12 CONN_01X04, J13 CONN_01X03, J14 CONN_01X03, J15 CONN_01X03, J16 CONN_01X03, J17 CONN_01X04, J2 CONN_01X08, J3 CONN_01X04, J4 CONN_01X03, J5 CONN_01X04, J6 CONN_01X03, J7 CONN_01X04, J8 CONN_01X04, J9 CONN_01X04, SW1 Rotary_Encoder, SW2 Rotary_Encoder, SW3 Rotary_Encoder, SW4 Rotary_Encoder, U1 MAX485CSA+, U2 ROE-0505S, U3 6N137, U4 Teensy3.5

Commit message: Silkscreen
Other:
- board text added: "1"
- board text added: "12V"
- board text added: "2"
- board text added: "3"
- board text added: "3V3"
- board text added: "4"
- board text added: "5V"
- board text added: "AUX"
- board text added: "BTN GND LED GND"
- board text added: "CLK"
- board text added: "CS"
- board text added: "Colordance v1.0"
- board text added: "DATA"
- board text added: "DMX"
- board text added: "GND"
- board text added: "GND BTN"
- board text added: "GND LED GND BTN"
- board text added: "I2C"
- board text added: "IN"
- board text added: "LED"
- board text added: "MIC"
- board text added: "MISO"
- board text added: "MOSI"
- board text added: "MOTION"
- board text added: "NEXT"
- board text added: "ON BTN"
- board text added: "ORIENTATION"
- board text added: "OUT"
- board text added: "POWER"
- board text added: "PREV"
- board text added: "RX"
- board text added: "SCK"
- board text added: "SCL"
- board text added: "SDA"
- board text added: "SPI"
- board text added: "SPI LED"
- board text added: "TEMPO"
- board text added: "TEST"
- board text added: "TX"
- board text added: "UART"
Changed lines of the file:
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@@
   (general
     (links 184)
-    (no_connects 1)
+    (no_connects 0)
     (area 20.949999 38.949999 201.050001 164.050001)
     (thickness 1.6)
-    (drawings 9)
+    (drawings 93)
     (tracks 681)
     (zones 0)
@@
   (page A3)
   (layers
-    (0 F.Cu signal)
-    (31 B.Cu signal)
+    (0 F.Cu signal hide)
+    (31 B.Cu signal hide)
     (32 B.Adhes user)
     (33 F.Adhes user)
@@
     (47 F.CrtYd user)
     (48 B.Fab user hide)
-    (49 F.Fab user)
+    (49 F.Fab user hide)
   )
   (setup
@@
       (solder_mask_margin 0.1))
   )
+  (gr_text TEST (at 144.5 115) (layer F.SilkS)
+    (effects (font (size 1.5 1.5) (thickness 0.3)))
+  )
+  (gr_circle (center 140 115) (end 140.5 115.5) (layer F.SilkS) (width 1.5))
+  (gr_text "Colordance v1.0" (at 98.5 112.5) (layer F.SilkS)
+    (effects (font (size 3 3) (thickness 0.5)))
+  )
+  (gr_text OUT (at 47.5 137) (layer B.SilkS)
+    (effects (font (size 1.2 1.2) (thickness 0.3)) (justify mirror))
+  )
+  (gr_text 3V3 (at 47.5 142) (layer B.SilkS)
+    (effects (font (size 1.2 1.2) (thickness 0.3)) (justify mirror))
+  )
+  (gr_text GND (at 47.5 144.5) (layer B.SilkS)
+    (effects (font (size 1.2 1.2) (thickness 0.3)) (justify mirror))
+  )
+  (gr_text DATA (at 65 149 90) (layer B.SilkS)
+    (effects (font (size 1.2 1.2) (thickness 0.3)) (justify mirror))
+  )
+  (gr_text CLK (at 61.5 149.5 90) (layer B.SilkS)
+    (effects (font (size 1.2 1.2) (thickness 0.3)) (justify mirror))
+  )
+  (gr_text 5V (at 58 150 90) (layer B.SilkS)
+    (effects (font (size 1.2 1.2) (thickness 0.3)) (justify mirror))
+  )
+  (gr_text GND (at 68.5 149.5 90) (layer B.SilkS)
+    (effects (font (size 1.2 1.2) (thickness 0.3)) (justify mirror))
+  )
+  (gr_text 12V (at 45.5 149.5 90) (layer B.SilkS)
+    (effects (font (size 1.2 1.2) (thickness 0.3)) (justify mirror))
+  )
+  (gr_text 5V (at 43 149.5 90) (layer B.SilkS)
+    (effects (font (size 1.2 1.2) (thickness 0.3)) (justify mirror))
+  )
+  (gr_text GND (at 40.5 149.5 90) (layer B.SilkS)
+    (effects (font (size 1.2 1.2) (thickness 0.3)) (justify mirror))
+  )
+  (gr_text GND (at 106.5 161.5) (layer B.SilkS)
+    (effects (font (size 1.5 1.5) (thickness 0.3)) (justify mirror))
+  )
+  (gr_text IN (at 105.5 159) (layer B.SilkS)
+    (effects (font (size 1.5 1.5) (thickness 0.3)) (justify mirror))
+  )
+  (gr_text 5V (at 105.5 156.5) (layer B.SilkS)
+    (effects (font (size 1.5 1.5) (thickness 0.3)) (justify mirror))
+  )
+  (gr_text IN (at 77.5 159) (layer B.SilkS)
+    (effects (font (size 1.5 1.5) (thickness 0.3)) (justify mirror))
+  )
+  (gr_text GND (at 76 161.5) (layer B.SilkS)
+    (effects (font (size 1.5 1.5) (thickness 0.3)) (justify mirror))
+  )
+  (gr_text 5V (at 77 156.5) (layer B.SilkS)
+    (effects (font (size 1.5 1.5) (thickness 0.3)) (justify mirror))
+  )
+  (gr_text CS (at 153.5 159) (layer B.SilkS)
+    (effects (font (size 1.5 1.5) (thickness 0.3)) (justify mirror))
+  )
+  (gr_text MOSI (at 154.5 156.5) (layer B.SilkS)
+    (effects (font (size 1.5 1.5) (thickness 0.3)) (justify mirror))
+  )
+  (gr_text MISO (at 154.5 154) (layer B.SilkS)
+    (effects (font (size 1.5 1.5) (thickness 0.3)) (justify mirror))
+  )
+  (gr_text SCK (at 154 151.5) (layer B.SilkS)
+    (effects (font (size 1.5 1.5) (thickness 0.3)) (justify mirror))
+  )
+  (gr_text MIC (at 139 159) (layer B.SilkS)
+    (effects (font (size 1.5 1.5) (thickness 0.3)) (justify mirror))
+  )
+  (gr_text RX (at 132 159) (layer B.SilkS)
+    (effects (font (size 1.5 1.5) (thickness 0.3)) (justify mirror))
+  )
+  (gr_text TX (at 132 156.5) (layer B.SilkS)
+    (effects (font (size 1.5 1.5) (thickness 0.3)) (justify mirror))
+  )
+  (gr_text 2 (at 125 159) (layer B.SilkS)
+    (effects (font (size 1.5 1.5) (thickness 0.3)) (justify mirror))
+  )
+  (gr_text 1 (at 125 156) (layer B.SilkS)
+    (effects (font (size 1.5 1.5) (thickness 0.3)) (justify mirror))
+  )
+  (gr_text SCL (at 116.5 159) (layer B.SilkS)
+    (effects (font (size 1.5 1.5) (thickness 0.3)) (justify mirror))
+  )
+  (gr_text SDA (at 116.5 156.5) (layer B.SilkS)
+    (effects (font (size 1.5 1.5) (thickness 0.3)) (justify mirror))
+  )
+  (gr_line (start 151 149) (end 152 149) (layer B.SilkS) (width 0.2))
+  (gr_text 3V3 (at 154 149) (layer B.SilkS)
+    (effects (font (size 1.5 1.5) (thickness 0.3)) (justify mirror))
+  )
+  (gr_line (start 143.5 156.5) (end 149 149) (layer B.SilkS) (width 0.2))
+  (gr_line (start 136 154) (end 141.5 156.5) (layer B.SilkS) (width 0.2))
+  (gr_line (start 128.5 154) (end 134 154) (layer B.SilkS) (width 0.2))
+  (gr_line (start 121 154) (end 126.5 154) (layer B.SilkS) (width 0.2))
+  (gr_line (start 118 154) (end 119 154) (layer B.SilkS) (width 0.2))
+  (gr_text 3V3 (at 116 154) (layer B.SilkS)
+    (effects (font (size 1.5 1.5) (thickness 0.3)) (justify mirror))
+  )
+  (gr_text I2C (at 120 151) (layer B.SilkS)
+    (effects (font (size 1.5 1.5) (thickness 0.3)) (justify mirror))
+  )
+  (gr_text AUX (at 127.5 151) (layer B.SilkS)
+    (effects (font (size 1.5 1.5) (thickness 0.3)) (justify mirror))
+  )
+  (gr_text UART (at 135 151) (layer B.SilkS)
+    (effects (font (size 1.5 1.5) (thickness 0.3)) (justify mirror))
+  )
+  (gr_text MIC (at 142.5 153.5) (layer B.SilkS)
+    (effects (font (size 1.5 1.5) (thickness 0.3)) (justify mirror))
+  )
+  (gr_text SPI (at 150 146) (layer B.SilkS)
+    (effects (font (size 1.5 1.5) (thickness 0.3)) (justify mirror))
+  )
+  (gr_line (start 119 161.5) (end 118.5 161.5) (layer B.SilkS) (width 0.2))
+  (gr_line (start 151 161.5) (end 151.5 161.5) (layer B.SilkS) (width 0.2))
+  (gr_line (start 143.5 161.5) (end 149 161.5) (layer B.SilkS) (width 0.2))
+  (gr_line (start 136 161.5) (end 141.5 161.5) (layer B.SilkS) (width 0.2))
+  (gr_line (start 129 161.5) (end 134 161.5) (layer B.SilkS) (width 0.2))
+  (gr_line (start 121 161.5) (end 126.5 161.5) (layer B.SilkS) (width 0.2))
+  (gr_text GND (at 116 161.5) (layer B.SilkS)
+    (effects (font (size 1.5 1.5) (thickness 0.3)) (justify mirror))
+  )
+  (gr_text GND (at 154 161.5) (layer B.SilkS)
+    (effects (font (size 1.5 1.5) (thickness 0.3)) (justify mirror))
+  )
+  (gr_line (start 80 152) (end 102.5 152) (layer B.SilkS) (width 0.2))
+  (gr_text 1 (at 80 153.5) (layer B.SilkS)
+    (effects (font (size 1.5 1.5) (thickness 0.3)) (justify mirror))
+  )
+  (gr_text 2 (at 87.5 153.5) (layer B.SilkS)
+    (effects (font (size 1.5 1.5) (thickness 0.3)) (justify mirror))
+  )
+  (gr_text 3 (at 95 153.5) (layer B.SilkS)
+    (effects (font (size 1.5 1.5) (thickness 0.3)) (justify mirror))
+  )
+  (gr_text 4 (at 102.5 153.5) (layer B.SilkS)
+    (effects (font (size 1.5 1.5) (thickness 0.3)) (justify mirror))
+  )
+  (gr_text MOTION (at 91 149.5) (layer B.SilkS)
+    (effects (font (size 2 2) (thickness 0.3)) (justify mirror))
+  )
+  (gr_line (start 183.5 109.5) (end 183.5 118.5) (layer B.SilkS) (width 0.2))
+  (gr_line (start 183.5 70.5) (end 183.5 79) (layer B.SilkS) (width 0.2))
+  (gr_line (start 183.5 56) (end 183.5 64.5) (layer B.SilkS) (width 0.2))
+  (gr_text NEXT (at 180.5 60.5 90) (layer B.SilkS)
+    (effects (font (size 2 2) (thickness 0.3)) (justify mirror))
+  )
+  (gr_text PREV (at 180.5 75 90) (layer B.SilkS)
+    (effects (font (size 2 2) (thickness 0.3)) (justify mirror))
+  )
+  (gr_text "ON BTN" (at 193 103.5) (layer B.SilkS)
+    (effects (font (size 2 2) (thickness 0.3)) (justify mirror))
+  )
+  (gr_text "SPI LED" (at 54.5 158 90) (layer B.SilkS)
+    (effects (font (size 2 2) (thickness 0.3)) (justify mirror))
+  )
+  (gr_text POWER (at 35 158 90) (layer B.SilkS)
+    (effects (font (size 2 2) (thickness 0.3)) (justify mirror))
+  )
+  (gr_line (start 42.5 124.5) (end 42.5 133.5) (layer B.SilkS) (width 0.2))
+  (gr_line (start 42.5 104) (end 42.5 112.5) (layer B.SilkS) (width 0.2))
+  (gr_text TEMPO (at 49 129) (layer B.SilkS)
+    (effects (font (size 2 2) (thickness 0.3)) (justify mirror))
+  )
+  (gr_text ORIENTATION (at 53.5 108) (layer B.SilkS)
+    (effects (font (size 2 2) (thickness 0.3)) (justify mirror))
+  )
+  (gr_text "BTN\nGND\nLED\nGND" (at 186 60.5) (layer B.SilkS)
+    (effects (font (size 1.5 1.5) (thickness 0.3)) (justify mirror))
+  )
+  (gr_text "BTN\nGND\nLED\nGND" (at 186 75) (layer B.SilkS)
+    (effects (font (size 1.5 1.5) (thickness 0.3)) (justify mirror))
+  )
+  (gr_text "BTN\nGND\nLED\nGND" (at 186 114) (layer B.SilkS)
+    (effects (font (size 1.5 1.5) (thickness 0.3)) (justify mirror))
+  )
+  (gr_text "GND\nLED\nGND\nBTN" (at 40 129) (layer B.SilkS)
+    (effects (font (size 1.5 1.5) (thickness 0.3)) (justify mirror))
+  )
+  (gr_text "GND\nBTN" (at 40 110.5) (layer B.SilkS)
+    (effects (font (size 1.5 1.5) (thickness 0.3)) (justify mirror))
+  )
+  (gr_text LED (at 40 107) (layer B.SilkS)
+    (effects (font (size 1.5 1.5) (thickness 0.3)) (justify mirror))
+  )
+  (gr_text GND (at 40 104.5) (layer B.SilkS)
+    (effects (font (size 1.5 1.5) (thickness 0.3)) (justify mirror))
+  )
+  (gr_text NEXT (at 199 61 90) (layer F.SilkS)
+    (effects (font (size 1.5 1.5) (thickness 0.3)))
+  )
+  (gr_text PREV (at 199 75 90) (layer F.SilkS)
+    (effects (font (size 1.5 1.5) (thickness 0.3)))
+  )
+  (gr_text "ON BTN" (at 199.5 113 90) (layer F.SilkS)
+    (effects (font (size 1.5 1.5) (thickness 0.3)))
+  )
+  (gr_text DMX (at 172 162.5) (layer F.SilkS)
+    (effects (font (size 1.5 1.5) (thickness 0.3)))
+  )
+  (gr_text "SPI LED" (at 64 162.5) (layer F.SilkS)
+    (effects (font (size 1.5 1.5) (thickness 0.3)))
+  )
+  (gr_text POWER (at 44 162.5) (layer F.SilkS)
+    (effects (font (size 1.5 1.5) (thickness 0.3)))
+  )
+  (gr_text ORIENTATION (at 26 111 270) (layer F.SilkS)
+    (effects (font (size 1.5 1.5) (thickness 0.3)))
+  )
+  (gr_text TEMPO (at 26 129.5 270) (layer F.SilkS)
+    (effects (font (size 1.5 1.5) (thickness 0.3)))
+  )
   (gr_line (start 21 164) (end 21 39) (layer Edge.Cuts) (width 0.1))
