File: colordance_mini.sch (KiCad schematic (older format))
At the start: 75 parts, among them J1 XLR3, J10 CONN_01X06, J11 CONN_01X04, J12 CONN_01X04, J13 CONN_01X03, J14 CONN_01X03, J15 CONN_01X03, J16 CONN_01X03, J17 CONN_01X04, J2 CONN_01X08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

Commit message: Revision 1.1
- Fix Teensy footprint to not use pads
- Opto isolator gets 3v3 instead of 5v
- Separate ground for DMX side
- Fix DMX connector pinout
Parts:
- U4: footprint teensy:Teensy35_36 -> homebrew:Teensy35_36; symbol Teensy3.5-RESCUE-colordance_mini -> Teensy3.5_simple
Connections:
- net +3V3: now also U3.2 (A), U4.15 (3.3V); no longer U4.75 (3.3V)
- net +5V: no longer U3.2 (A)
- net AUX_CS: now also U4.42 (15_A1_CS0_Touch); no longer U4.70 (43_CS2)
- net AUX_MISO: now also U4.14 (12_MISO0); no longer U4.72 (45_MISO2)
- net AUX_MOSI: now also U4.13 (11_MOSI0); no longer U4.71 (44_MOSI2)
- net AUX_SCK: now also U4.40 (13_SCK0_LED); no longer U4.73 (46_SCK2)
- net DENSITY: now also U4.38 (A22_DAC1); no longer U4.45 (18_A4_SDA0_Touch)
- net GND: no longer C7.2, C8.2, J1.1, R5.2, U1.5 (GND), U2.3 (-VOUT), U3.5 (GND)
- net MOTION_1: now also U4.3 (1_TX1_MISO1_Touch); no longer U4.86 (57)
- net MOTION_2: now also U4.23 (31_A12_RX4_CS1); no longer U4.85 (56)
- net MOTION_3: now also U4.56 (A10); no longer U4.84 (55)
- net MOTION_4: now also U4.57 (A11); no longer U4.83 (54_CS2)
- net ORIENTATION: now also U4.31 (34_A15_CAN1TX_sda0); no longer U4.13 (11_MOSI0)
- net PARAM: now also U4.37 (A21_DAC0); no longer U4.46 (19_A5_SCL0_Touch)
- net SCL0: now also U4.46 (19_A5_SCL0_Touch); no longer U4.76 (47_RX6_SCL0)
- net SDA0: now also U4.45 (18_A4_SDA0_Touch); no longer U4.77 (48_TX6_SDA0)
- net TEMPO_TAP: now also U4.36 (39_A20); no longer U4.14 (12_MISO0)
- net TILT: now also U4.50 (23_A9_PWM_Touch); no longer U4.42 (15_A1_CS0_Touch)
- net at R4.2, U1.6 (A): now also J1.3, R1.2; no longer J1.2, R1.1
- net at R5.1, U1.7 (B): now also J1.2, R1.1; no longer J1.3, R1.2
- new net GND_DMX: C7.2, C8.2, J1.1, R5.2, U1.5 (GND), U2.3 (-VOUT), U3.5 (GND)
- no-connect marks 37 -> 13
