File: colordance_mini.sch (KiCad schematic (older format))
At the start: 75 parts, among them J1 XLR3, J10 CONN_01X06, J11 CONN_01X04, J12 CONN_01X04, J13 CONN_01X03, J14 CONN_01X03, J15 CONN_01X03, J16 CONN_01X03, J17 CONN_01X04, J2 CONN_01X08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

Commit message: Hardware revision v1.2:
- Switch power to Anderson connector
- Switch SPI LED connector to soldered 4-pin JST
- Add filter caps to the pots
- Add a few decoupling caps
Parts:
- removed J4: CONN_01X03, homebrew:1985218_phoenix_4pos_3.5mm, symbol colordance_mini-rescue:CONN_01X03
- removed R2: 3k3, Resistors_SMD:R_0603_HandSoldering, symbol colordance_mini-rescue:R
- removed R3: 1k, Resistors_SMD:R_0603_HandSoldering, symbol colordance_mini-rescue:R
- added BT1: BATTERY-20MM_SMD, Sparkfun-Batteries:BATTCON_20MM, symbol SparkFun-Batteries:BATTERY-20MM_SMD
- added C15, C16, C17, C18, C19, C20: .1uF, Capacitor_SMD:C_0603_1608Metric_Pad1.05x0.95mm_HandSolder, symbol colordance_mini-rescue:C
- added C21, C22, C23: 1uF, Capacitor_SMD:C_0603_1608Metric_Pad1.05x0.95mm_HandSolder, symbol colordance_mini-rescue:C
- added J4: Anderson_two_redblack, homebrew:Anderson_1337G3_straight_two, symbol homebrew:Anderson_two_redblack
- J3: footprint homebrew:1985218_phoenix_4pos_3.5mm -> Connector_PinHeader_2.54mm:PinHeader_1x04_P2.54mm_Vertical
Connections:
- net +5V: now also C22.1, C23.1, J4.1
- net DENSITY: now also C19.1
- net GND: now also BT1.2 (-), C15.2, C16.2, C17.2, C18.2, C19.2, C20.2, C22.2, C23.2, J4.2
- net GND_DMX: now also C21.2
- net HEIGHT: now also C16.1
- net PAN: now also C17.1
- net PARAM: now also C20.1
- net TILT: now also C15.1
- net VDMX: now also C21.1
- net WIDTH: now also C18.1
- net at U4.25 (VBat): now also BT1.1 (+)
- net at J3.2 (P2): now also D1.6 (DO); no longer D1.5 (CO)
- net at J3.3 (P3): now also D1.5 (CO); no longer D1.6 (DO)
- net VBATT_DIV: no longer names the net of U4.48 (21_A7_PWM_CS0_sck1)
Other:
- note removed: "Battery voltage monitor"
- moved on the sheet: J3, RV2, RV3, RV4, RV5, RV6
